Commit message: 改为使用gazebo classic11仿真

File: src/agv_sim/description/robot.urdf.xacro (robot description, xacro)
@@ -2,10 +2,25 @@
 <robot xmlns:xacro="http://www.ros.org/wiki/xacro" name="robot">
     <xacro:arg name="use_ros2_control" default="true"/>
+    <xacro:arg name="robot_namespace" default="agv_sim"/>
     <!-- robot description -->
     <xacro:include filename="robot_core.xacro" />
-    <!-- use ros2_control -->
+    <!-- 机械臂 -->
+    <!-- <xacro:include filename="$(find my_arm)/config/panda.urdf.xacro" /> -->
+    <!-- <xacro:include filename="$(find moveit_resources_panda_description)/urdf/panda.urdf" />
+    <joint name="arm_joint" type="fixed">
+        <parent link="base_link" />
+        <child link = "panda_link0" />
+        <origin xyz="0.0 0.0 0.0" rpy="0.0 0.0 0.0" />
+    </joint> -->
+    <!-- 车轮控制器 -->
     <xacro:include filename="$(find agv_sim)/description/ros2_control.xacro" />
     <xacro:agv_sim_ros2_control />
-    <xacro:include filename="$(find agv_sim)/description/ign.xacro"/>
+    <!-- 机械臂控制器 -->
+    <!-- <xacro:include filename="$(find my_arm)/config/panda.ros2_control.xacro" /> -->
+    <!-- ign 仿真配置 -->
+    <!-- <xacro:include filename="$(find agv_sim)/description/ign.xacro"/> -->
+    <!-- gazebo 仿真配置 -->
+    <xacro:include filename="$(find agv_sim)/description/gazebo.xacro"/>
+    <xacro:gazebo_sensor />
     <!-- unless ros2_control, use gazebo_control -->
     <!-- <xacro:unless value="$(arg use_ros2_control)">

File: src/agv_sim/description/robot_core.xacro (robot description, xacro)
@@ -30,7 +30,4 @@
     <xacro:arg name="robot_namespace" default=""/>
     <xacro:arg name="wheel_odom_topic" default="odom" />
-    <xacro:arg name="camera_enabled" default="false" />
-    <xacro:arg name="stereo_camera_enabled" default="false" />
-    <xacro:arg name="two_d_lidar_enabled" default="false" />
     <xacro:arg name="publish_wheel_odom_tf" default="true" />
     <xacro:arg name="conveyor_enabled" default="false"/>
@@ -81,34 +78,32 @@
     <xacro:traction_wheel cardinality="middle" dexterity="right" origin_x="0" origin_y="-${traction_track_width/2}" origin_z="-${chassis_height/2+2*trolley_wheel_radius+eps-traction_wheel_radius}"/>
     <!-- ............................. 2D LIDAR ........................................ -->
-    <xacro:if value="$(arg two_d_lidar_enabled)">
-        <link name="two_d_lidar">
-            <collision>
-                <origin xyz="0 0 0" rpy="0 0 0" />
-                <geometry>
-                    <cylinder length="0.06" radius="0.075"/>
-                </geometry>
-            </collision>
-            <visual>
-                <origin xyz="0 0 0" rpy="0 0 0" />
-                <geometry>
-                    <cylinder length="0.06" radius="0.075"/>
-                </geometry>
-                <material name="aluminium"/>
-            </visual>
-            <inertial>
-                <origin xyz="0 0 0" rpy="0 0 0" />
-                <mass value="0.1"/>
-                <xacro:cylinder_inertia m="0.1" r="0.075" h="0.06"/>
-            </inertial>
-        </link>
-        <joint name="two_d_lidar_joint" type="fixed">
-            <parent link="base_link"/>
-            <child link="two_d_lidar"/>
-            <origin xyz="0.0 0 0.08" rpy="0 0 0" />
-        </joint>
-        <gazebo reference="two_d_lidar">
-            <material>Gazebo/White</material>
-        </gazebo>
-    </xacro:if>
+    <link name="two_d_lidar">
+        <collision>
+            <origin xyz="0 0 0" rpy="0 0 0" />
+            <geometry>
+                <cylinder length="0.06" radius="0.075"/>
+            </geometry>
+        </collision>
+        <visual>
+            <origin xyz="0 0 0" rpy="0 0 0" />
+            <geometry>
+                <cylinder length="0.06" radius="0.075"/>
+            </geometry>
+            <material name="aluminium"/>
+        </visual>
+        <inertial>
+            <origin xyz="0 0 0" rpy="0 0 0" />
+            <mass value="0.1"/>
+            <xacro:cylinder_inertia m="0.1" r="0.075" h="0.06"/>
+        </inertial>
+    </link>
+    <joint name="two_d_lidar_joint" type="fixed">
+        <parent link="base_link"/>
+        <child link="two_d_lidar"/>
+        <origin xyz="0.0 0 0.08" rpy="0 0 0" />
+    </joint>
+    <gazebo reference="two_d_lidar">
+        <material>Gazebo/White</material>
+    </gazebo>
     <!-- ............................. IMU ........................................ -->
     <link name="imu_frame"/>
@@ -119,71 +114,67 @@
     </joint>
     <!-- ............................. CAMERA ........................................ -->
-    <xacro:if value="$(arg camera_enabled)">
-        <!-- KINECT CAMERA -->
-        <link name="kinect_camera">
-            <collision>
-                <origin xyz="0 0 0" rpy="0 0 0" />
-                <geometry>
-                    <box size="0.07 0.3 0.09"/>
-                </geometry>
-            </collision>
-            <visual>
-                <origin xyz="0 0 0" rpy="0 0 0" />
-                <geometry>
-                    <mesh filename="file://$(find agv_sim)/meshes/kinect/d415.dae"/>
-                </geometry>
-                <material name="black"/>
-            </visual>
-            <inertial>
-                <mass value="0.01"/>
-                <xacro:box_inertia m="0.01" x="0.07" y="0.3" z = "0.09"/>
-            </inertial>
-        </link>
-        <joint name="kinect_camera_joint" type="fixed">
-            <origin rpy="0 0 0" xyz="${chassis_length/2} 0 ${chassis_height/7}"/>
-            <parent link="base_link"/>
-            <child link="kinect_camera"/>
-        </joint>
-        <link name="kinect_camera_optical"/>
-        <joint name="kinect_camera_optical_joint" type="fixed">
-            <origin xyz="0 0 0" rpy="${-pi/2} 0 ${-pi/2}"/>
-            <parent link="kinect_camera"/>
-            <child link="kinect_camera_optical"/>
-        </joint>
-    </xacro:if>
+    <!-- KINECT CAMERA -->
+    <link name="kinect_camera">
+        <collision>
+            <origin xyz="0 0 0" rpy="0 0 0" />
+            <geometry>
+                <box size="0.07 0.3 0.09"/>
+            </geometry>
+        </collision>
+        <visual>
+            <origin xyz="0 0 0" rpy="0 0 0" />
+            <geometry>
+                <mesh filename="file://$(find agv_sim)/meshes/kinect/d415.dae"/>
+            </geometry>
+            <material name="black"/>
+        </visual>
+        <inertial>
+            <mass value="0.01"/>
+            <xacro:box_inertia m="0.01" x="0.07" y="0.3" z = "0.09"/>
+        </inertial>
+    </link>
+    <joint name="kinect_camera_joint" type="fixed">
+        <origin rpy="0 0 0" xyz="${chassis_length/2} 0 ${chassis_height/7}"/>
+        <parent link="base_link"/>
+        <child link="kinect_camera"/>
+    </joint>
+    <link name="kinect_camera_optical"/>
+    <joint name="kinect_camera_optical_joint" type="fixed">
+        <origin xyz="0 0 0" rpy="${-pi/2} 0 ${-pi/2}"/>
+        <parent link="kinect_camera"/>
+        <child link="kinect_camera_optical"/>
+    </joint>
     <!-- .............................STEREO CAMERA ........................................ -->
-    <xacro:if value="$(arg stereo_camera_enabled)">
-        <!-- STEREO CAMERA -->
-        <link name="stereo_camera">
-            <collision>
-                <origin xyz="0 0 0" rpy="0 0 0" />
-                <geometry>
-                    <box size="0.07 0.3 0.09"/>
-                </geometry>
-            </collision>
-            <visual>
-                <origin xyz="0 0 0" rpy="0 0 0" />
-                <geometry>
-                    <mesh filename="file://$(find agv_sim)/meshes/kinect/d415.dae"/>
-                </geometry>
-                <material name="black"/>
-            </visual>
-            <inertial>
-                <mass value="0.01"/>
-                <xacro:box_inertia m="0.01" x="0.07" y="0.3" z = "0.09"/>
-            </inertial>
-        </link>
-        <joint name="stereo_camera_joint" type="fixed">
-            <origin rpy="0 0 0" xyz="${chassis_length/2} 0 ${chassis_height/7}"/>
-            <parent link="base_link"/>
-            <child link="stereo_camera"/>
-        </joint>
-        <link name="stereo_camera_optical"/>
-        <joint name="stereo_camera_optical_joint" type="fixed">
-            <origin xyz="0 0 0" rpy="${-pi/2} 0 ${-pi/2}"/>
-            <parent link="stereo_camera"/>
-            <child link="stereo_camera_optical"/>
-        </joint>
-    </xacro:if>
+    <!-- STEREO CAMERA -->
+    <link name="stereo_camera">
+        <collision>
+            <origin xyz="0 0 0" rpy="0 0 0" />
+            <geometry>
+                <box size="0.07 0.3 0.09"/>
+            </geometry>
+        </collision>
+        <visual>
+            <origin xyz="0 0 0" rpy="0 0 0" />
+            <geometry>
+                <mesh filename="file://$(find agv_sim)/meshes/kinect/d415.dae"/>
+            </geometry>
+            <material name="black"/>
+        </visual>
+        <inertial>
+            <mass value="0.01"/>
+            <xacro:box_inertia m="0.01" x="0.07" y="0.3" z = "0.09"/>
+        </inertial>
+    </link>
+    <joint name="stereo_camera_joint" type="fixed">
+        <origin rpy="0 0 0" xyz="${chassis_length/2} 0 ${chassis_height/7}"/>
+        <parent link="base_link"/>
+        <child link="stereo_camera"/>
+    </joint>
+    <link name="stereo_camera_optical"/>
+    <joint name="stereo_camera_optical_joint" type="fixed">
+        <origin xyz="0 0 0" rpy="${-pi/2} 0 ${-pi/2}"/>
+        <parent link="stereo_camera"/>
+        <child link="stereo_camera_optical"/>
+    </joint>
     <!-- ............................. ROOF ........................................ -->
     <link name="roof_link">

File: src/agv_sim/description/ros2_control.xacro (robot description, xacro)
@@ -2,7 +2,8 @@
 <robot xmlns:xacro="http://www.ros.org/wiki/xacro">
     <xacro:macro name="agv_sim_ros2_control">
-        <ros2_control name="AgvSimGazeboSystem" type="system">
+        <ros2_control name="GazeboSystem" type="system">
             <hardware>
-                <plugin>ign_ros2_control/IgnitionSystem</plugin>
+                <!-- <plugin>ign_ros2_control/IgnitionSystem</plugin> -->
+                <plugin>gazebo_ros2_control/GazeboSystem</plugin>
             </hardware>
             <joint name="middle_left_wheel_joint">
@@ -24,6 +25,13 @@
         </ros2_control>
         <gazebo>
-            <plugin filename="ign_ros2_control-system" name="ign_ros2_control::IgnitionROS2ControlPlugin">
-                <parameters>$(find agv_sim)/config/ros2_controller.yaml</parameters>
+            <!-- <plugin filename="ign_ros2_control-system" name="ign_ros2_control::IgnitionROS2ControlPlugin">
+                <parameters>$(find bcr_bot)/config/ros2_controller.yaml</parameters>
+                <ros>
+                    <remapping>/diff_drive_controller/cmd_vel_unstamped:=/cmd_vel</remapping>
+                    <remapping>/diff_drive_controller/odom:=/odom</remapping>
+                </ros>
+            </plugin> -->
+            <plugin name="gazebo_ros2_control" filename="libgazebo_ros2_control.so">
+                <parameters>$(find bcr_bot)/config/ros2_controller.yaml</parameters>
                 <ros>
                     <remapping>/diff_drive_controller/cmd_vel_unstamped:=/cmd_vel</remapping>
