Commit message: 通过设置arm_enable来启用或者不启用机械臂

File: src/agv_with_arm/urdf/agv/macros.xacro (robot description, xacro)
@@ -25,5 +25,5 @@
                 <xacro:sphere_inertia m="${trolley_wheel_mass}" r="${trolley_wheel_radius}"/>
             </inertial>
-            <mu>0.0</mu>
+            <mu>5.0</mu>
         </link>
         <joint name="${cardinality}_${dexterity}_wheel_joint" type="fixed">
@@ -45,4 +45,23 @@
                 </geometry>
                 <self_collide>false</self_collide>
+                <!-- 添加表面接触属性来模拟压力变形 -->
+                <surface>
+                    <contact>
+                        <ode>
+                            <kp>50000.0</kp>                            <!-- 弹簧刚度系数，用于模拟轮子和地面接触时的变形 -->
+                            <kd>1.0</kd>                            <!-- 阻尼系数，用于抑制快速变形 -->
+                            <erp>0.2</erp>                            <!-- 误差修正参数，表示接触的恢复率 -->
+                            <cfm>0.001</cfm>                            <!-- 约束力混合参数，表示柔性程度 -->
+                        </ode>
+                    </contact>
+                    <friction>
+                        <ode>
+                            <mu>10.0</mu>                            <!-- 主摩擦系数 -->
+                            <mu2>5.0</mu2>                            <!-- 次摩擦系数 -->
+                            <slip1>0.01</slip1>                            <!-- 在主方向的滑动 -->
+                            <slip2>0.01</slip2>                            <!-- 在次方向的滑动 -->
+                        </ode>
+                    </friction>
+                </surface>
             </collision>
             <inertial>
@@ -51,5 +70,5 @@
                 <xacro:cylinder_inertia m="${traction_wheel_mass}" r="${traction_wheel_radius}" h="${traction_wheel_width}"/>
             </inertial>
-            <mu>5.0</mu>
+            <mu>10.0</mu>
         </link>
         <joint name="${cardinality}_${dexterity}_wheel_joint" type="continuous">

File: src/agv_with_arm/urdf/agv/robot.urdf.xacro (robot description, xacro)
@@ -1,21 +1,20 @@
 <?xml version="1.0"?>
 <robot xmlns:xacro="http://www.ros.org/wiki/xacro" name="robot">
-    <xacro:arg name="use_ros2_control" default="true"/>
+    <xacro:arg name="arm_enabled" default="true"/>
     <xacro:arg name="robot_namespace" default="agv_with_arm"/>
     <!-- robot description -->
     <xacro:include filename="robot_core.xacro" />
     <!-- 机械臂 -->
-    <!-- <xacro:include filename="$(find my_arm)/config/panda.urdf.xacro" /> -->
-    <!-- <xacro:include filename="$(find moveit_resources_panda_description)/urdf/panda.urdf" />
-    <joint name="arm_joint" type="fixed">
-        <parent link="base_link" />
-        <child link = "panda_link0" />
-        <origin xyz="0.0 0.0 0.0" rpy="0.0 0.0 0.0" />
-    </joint> -->
-    <!-- 车轮控制器 -->
+    <xacro:if value="$(arg arm_enabled)">
+        <xacro:include filename="$(find agv_with_arm)/urdf/arm/aubo.gazebo.xacro" />
+        <joint name="arm_joint" type="fixed">
+            <parent link="roof_link" />
+            <child link = "arm_base_link" />
+            <origin xyz="0.0 0.0 0.0" rpy="0.0 0.0 0.0" />
+        </joint>
+    </xacro:if>
+    <!-- 控制器 -->
     <xacro:include filename="$(find agv_with_arm)/urdf/agv/ros2_control.xacro" />
-    <xacro:agv_sim_ros2_control />
-    <!-- 机械臂控制器 -->
-    <!-- <xacro:include filename="$(find my_arm)/config/panda.ros2_control.xacro" /> -->
+    <xacro:agv_sim_ros2_control arm_enabled="$(arg arm_enabled)"/>
     <!-- gazebo 仿真配置 -->
     <xacro:include filename="$(find agv_with_arm)/urdf/agv/gazebo_sensor.xacro"/>

File: src/agv_with_arm/urdf/agv/robot_core.xacro (robot description, xacro)
@@ -2,5 +2,5 @@
 <robot xmlns:xacro="http://www.ros.org/wiki/xacro" name="agv_with_arm">
     <!--................................ XACRO CONSTANTS .............................. -->
-    <xacro:property name="chassis_mass" value="70"/>
+    <xacro:property name="chassis_mass" value="5"/>
     <xacro:property name="chassis_length" value="0.9"/>
     <xacro:property name="chassis_width" value="0.64"/>
@@ -15,5 +15,5 @@
     <xacro:property name="trolley_wheel_radius" value="0.06"/>
     <!-- a small constant -->
-    <xacro:property name="eps" value="0.002"/>
+    <xacro:property name="eps" value="0.001"/>
     <xacro:property name="traction_wheel_radius" value="0.1"/>
     <xacro:property name="traction_wheel_width" value="0.05"/>

File: src/agv_with_arm/urdf/agv/ros2_control.xacro (robot description, xacro)
@@ -1,5 +1,5 @@
 <?xml version="1.0"?>
 <robot xmlns:xacro="http://www.ros.org/wiki/xacro">
-    <xacro:macro name="agv_sim_ros2_control">
+    <xacro:macro name="agv_sim_ros2_control" params="arm_enabled">
         <ros2_control name="GazeboSystem" type="system">
             <hardware>
@@ -22,7 +22,100 @@
                 <state_interface name="velocity" />
             </joint>
+            <!-- =================================================================== -->
+            <xacro:if value="${arm_enabled}">
+                <joint name="shoulder_joint">
+                    <command_interface name="position">
+                        <param name="min">${-2*pi}</param>
+                        <param name="max">${2*pi}</param>
+                    </command_interface>
+                    <command_interface name="velocity">follow_joint_trajectory
+                        <param name="min">-3.15</param>
+                        <param name="max">3.15</param>
+                    </command_interface>
+                    <state_interface name="position">
+                        <param name="initial_value">0.0</param>
+                    </state_interface>
+                    <state_interface name="velocity"/>
+                    <!-- <state_interface name="effort"/> -->
+                </joint>
+                <joint name="upperArm_joint">
+                    <command_interface name="position">
+                        <param name="min">${-2*pi}</param>
+                        <param name="max">${2*pi}</param>
+                    </command_interface>
+                    <command_interface name="velocity">
+                        <param name="min">-3.15</param>
+                        <param name="max">3.15</param>
+                    </command_interface>
+                    <state_interface name="position">
+                        <param name="initial_value">-1.57</param>
+                    </state_interface>
+                    <state_interface name="velocity"/>
+                    <!-- <state_interface name="effort"/> -->
+                </joint>
+                <joint name="foreArm_joint">
+                    <command_interface name="position">
+                        <param name="min">${-pi}</param>
+                        <param name="max">${pi}</param>
+                    </command_interface>
+                    <command_interface name="velocity">
+                        <param name="min">-3.15</param>
+                        <param name="max">3.15</param>
+                    </command_interface>
+                    <state_interface name="position">
+                        <param name="initial_value">0.0</param>
+                    </state_interface>
+                    <state_interface name="velocity"/>
+                    <!-- <state_interface name="effort"/> -->
+                </joint>
+                <joint name="wrist1_joint">
+                    <command_interface name="position">
+                        <param name="min">${-2*pi}</param>
+                        <param name="max">${2*pi}</param>
+                    </command_interface>
+                    <command_interface name="velocity">
+                        <param name="min">-6.28</param>
+                        <param name="max">6.28</param>
+                    </command_interface>
+                    <state_interface name="position">
+                        <param name="initial_value">0.0</param>
+                    </state_interface>
+                    <state_interface name="velocity"/>
+                    <!-- <state_interface name="effort"/> -->
+                </joint>
+                <joint name="wrist2_joint">
+                    <command_interface name="position">
+                        <param name="min">${-2*pi}</param>
+                        <param name="max">${2*pi}</param>
+                    </command_interface>
+                    <command_interface name="velocity">
+                        <param name="min">-6.28</param>
+                        <param name="max">6.28</param>
+                    </command_interface>
+                    <state_interface name="position">
+                        <param name="initial_value">0.0</param>
+                    </state_interface>
+                    <state_interface name="velocity"/>
+                    <!-- <state_interface name="effort"/> -->
+                </joint>
+                <joint name="wrist3_joint">
+                    <command_interface name="position">
+                        <param name="min">${-2*pi}</param>
+                        <param name="max">${2*pi}</param>
+                    </command_interface>
+                    <command_interface name="velocity">
+                        <param name="min">-6.28</param>
+                        <param name="max">6.28</param>
+                    </command_interface>
+                    <state_interface name="position">
+                        <param name="initial_value">0.0</param>
+                    </state_interface>
+                    <state_interface name="velocity"/>
+                    <!-- <state_interface name="effort"/> -->
+                </joint>
+            </xacro:if>
         </ros2_control>
         <gazebo>
-            <plugin name="gazebo_ros2_control" filename="libgazebo_ros2_control.so">
+            <plugin name="agv_gazebo_ros2_control" filename="libgazebo_ros2_control.so">
                 <parameters>$(find agv_with_arm)/config/agv_controller.yaml</parameters>
                 <ros>

File: src/agv_with_arm/urdf/arm/aubo.gazebo.xacro (robot description, xacro)
@@ -6,12 +6,12 @@
 <robot name="aubo_i5"
      xmlns:xacro="http://www.ros.org/wiki/xacro">
-     <xacro:include filename="$(find agv_with_arm)/urdf/arm/materials.xacro" />
-     <xacro:include filename="$(find agv_with_arm)/urdf/arm/gazebo_ros2control.xacro" />
-     <xacro:aubo_ros2control />
-     <link name="base_link">
+     <!-- <xacro:include filename="$(find agv_with_arm)/urdf/arm/materials.xacro" /> -->
+     <!-- <xacro:include filename="$(find agv_with_arm)/urdf/arm/gazebo_ros2control.xacro" />
+     <xacro:aubo_ros2control /> -->
+     <link name="arm_base_link">
           <inertial>
                <origin xyz="-1.4795E-13 0.0015384 0.020951" rpy="0 0 0" />
-               <mass value="0.83419" />
-               <inertia ixx="0.0014414" ixy="7.8809E-15" ixz="8.5328E-16" iyy="0.0013542" iyz="-1.4364E-05" izz="0.0024659" />
+               <mass value="0.0419" />
+               <inertia ixx="0" ixy="0" ixz="0" iyy="0" iyz="0" izz="0" />
           </inertial>
           <visual>
@@ -34,6 +34,6 @@
           <inertial>
                <origin xyz="3.2508868974735E-07 0.00534955349296065 -0.00883689325611056" rpy="0 0 0" />
-               <mass value="1.57658348693929" />
-               <inertia ixx="0.0040640448663128" ixy="0" ixz="0" iyy="0.00392863238466817" iyz="-0.000160151642851425" izz="0.0030869857349184" />
+               <mass value="0.07658348693929" />
+               <inertia ixx="0" ixy="0" ixz="0" iyy="0" iyz="0" izz="0" />
           </inertial>
           <visual>
@@ -55,5 +55,5 @@
      <joint name="shoulder_joint" type="revolute">
           <origin xyz="0 0 0.122" rpy="0 0 3.1416" />
-          <parent link="base_link" />
+          <parent link="arm_base_link" />
           <child link="shoulder_Link" />
           <axis xyz="0 0 1" />
@@ -63,6 +63,6 @@
           <inertial>
                <origin xyz="0.203996646979614 2.01304585036544E-10 0.0127641545395984" rpy="0 0 0" />
-               <mass value="4.04175782265494" />
-               <inertia ixx="0.00965399211106204" ixy="0" ixz="0" iyy="0.144993869035655" iyz="0" izz="0.142607184038966" />
+               <mass value="0.04175782265494" />
+               <inertia ixx="0" ixy="0" ixz="0" iyy="0" iyz="0" izz="0" />
           </inertial>
           <visual>
@@ -92,6 +92,6 @@
           <inertial>
                <origin xyz="0.188922115560337 6.78882434739072E-07 0.0981026740461557" rpy="0 0 0" />
-               <mass value="2.27145669098343" />
-               <inertia ixx="0.00214322284946289" ixy="0" ixz="-0.00073120631553383" iyy="0.0443926090878205" iyz="0" izz="0.0441273797128365" />
+               <mass value="0.07145669098343" />
+               <inertia ixx="0" ixy="0" ixz="0" iyy="0" iyz="0" izz="0" />
           </inertial>
           <visual>
@@ -121,6 +121,6 @@
           <inertial>
                <origin xyz="7.54205137428592E-07 0.0062481254331257 -0.00392367464072373" rpy="0 0 0" />
-               <mass value="0.500477539188764" />
-               <inertia ixx="0.00071194605962081" ixy="0" ixz="0" iyy="0.00040588242872958" iyz="-2.30808694377512E-05" izz="0.000685574004861334" />
+               <mass value="0.000477539188764" />
+               <inertia ixx="0" ixy="0" ixz="0" iyy="0" iyz="0" izz="0" />
           </inertial>
           <visual>
@@ -150,6 +150,6 @@
           <inertial>
                <origin xyz="-7.54207620578635E-07 -0.00624812542617262 -0.00392367464115684" rpy="0 0 0" />
-               <mass value="0.500477539245988" />
-               <inertia ixx="0.00071194605981829" ixy="0" ixz="0" iyy="0.000405882428755442" iyz="2.30808694515886E-05" izz="0.000685574005112107" />
+               <mass value="0.000477539245988" />
+               <inertia ixx="0" ixy="0" ixz="0" iyy="0" iyz="0" izz="0" />
           </inertial>
           <visual>
@@ -179,6 +179,6 @@
           <inertial>
                <origin xyz="3.92048778449938E-10 0.000175788057281467 -0.0213294490706684" rpy="0 0 0" />
-               <mass value="0.158309554874285" />
-               <inertia ixx="7.31376196034769E-05" ixy="0" ixz="0" iyy="7.19528188876563E-05" iyz="0" izz="0.000108772439051422" />
+               <mass value="0.058309554874285" />
+               <inertia ixx="0" ixy="0" ixz="0" iyy="0" iyz="0" izz="0" />
           </inertial>
           <visual>
@@ -205,9 +205,9 @@
           <limit lower="-6.28" upper="6.28" effort="10" velocity="1.5" />
      </joint>
-     <link name="world" />
+     <!-- <link name="world" />
      <joint name="world_joint" type="fixed">
           <parent link="world" />
-          <child link = "base_link" />
+          <child link = "arm_base_link" />
           <origin xyz="0.0 0.0 0.0" rpy="0.0 0.0 0.0" />
-     </joint>
+     </joint> -->
 </robot>

File: src/agv_with_arm/urdf/arm/gazebo_ros2control.xacro (robot description, xacro)
@@ -3,10 +3,10 @@
     <xacro:macro name="aubo_ros2control">
         <!-- ===== Gazebo ROS2_CONTROL plugin ===== -->
-        <gazebo>
-            <plugin filename="libgazebo_ros2_control.so" name="gazebo_ros2_control">
+        <!-- <gazebo>
+            <plugin filename="libgazebo_ros2_control.so" name="arm_gazebo_ros2_control">
                 <robot_sim_type>gazebo_ros2_control/GazeboSystem</robot_sim_type>
                 <parameters>$(find agv_with_arm)/config/aubo_controller.yaml</parameters>
             </plugin>
-        </gazebo>
+        </gazebo> -->
         <!-- ========== ROS2 CONTROL ========== -->
         <ros2_control name="GazeboSystem" type="system">
