Commit message: 添加nav2和mapping

File: src/agv_with_arm/urdf/agv/gazebo_sensor.xacro (robot description, xacro)
@@ -94,5 +94,5 @@
                         <width>1024</width>
                         <height>1024</height>
-                        <format>R8G8B8</format>
+                        <format>BGR8</format>
                     </image>
                     <clip>
@@ -120,5 +120,5 @@
                         <width>1024</width>
                         <height>1024</height>
-                        <format>R8G8B8</format>
+                        <format>BGR8</format>
                     </image>
                     <clip>

File: src/agv_with_arm/urdf/agv/robot_core.xacro (robot description, xacro)
@@ -2,9 +2,9 @@
 <robot xmlns:xacro="http://www.ros.org/wiki/xacro" name="agv_with_arm">
     <!--................................ XACRO CONSTANTS .............................. -->
-    <xacro:property name="chassis_mass" value="5"/>
+    <xacro:property name="chassis_mass" value="1"/>
     <xacro:property name="chassis_length" value="0.9"/>
     <xacro:property name="chassis_width" value="0.64"/>
     <xacro:property name="chassis_height" value="0.19"/>
-    <xacro:property name="traction_wheel_mass" value="1"/>
+    <xacro:property name="traction_wheel_mass" value="0.5"/>
     <xacro:property name="traction_wheel_base" value="0.88"/>
     <xacro:property name="traction_max_wheel_torque" value="20000"/>

Commit message: 改为使用gazebo自带的控制，不用ros2_control来控制小车

File: src/agv_with_arm/urdf/agv/gazebo_sensor.xacro (robot description, xacro)
@@ -4,4 +4,35 @@
         <gazebo>
             <static>false</static>
+        </gazebo>
+        <!-- .....................MULTI WHEEL DIFF DRIVE ................................... -->
+        <gazebo>
+            <plugin name="diff_drive" filename="libgazebo_ros_diff_drive.so">
+                <ros>
+                    <remapping>cmd_vel:=cmd_vel</remapping>
+                    <remapping>odom:=odom</remapping>
+                </ros>
+                <legacy_mode>false</legacy_mode>
+                <update_rate>50.0</update_rate>
+                <left_joint>middle_left_wheel_joint</left_joint>
+                <right_joint>middle_right_wheel_joint</right_joint>
+                <wheel_separation>${traction_track_width+traction_wheel_width-0.01}</wheel_separation>
+                <wheel_diameter>${2*traction_wheel_radius+0.01}</wheel_diameter>
+                <robot_base_frame>base_footprint</robot_base_frame>
+                <max_wheel_torque>${traction_max_wheel_torque}</max_wheel_torque>
+                <command_topic>cmd_vel</command_topic>
+                <odometry_topic>$(arg wheel_odom_topic)</odometry_topic>
+                <odometry_frame>odom</odometry_frame>
+                <publish_odom_tf>$(arg publish_wheel_odom_tf)</publish_odom_tf>
+                <publish_wheel_tf>true</publish_wheel_tf>
+                <publish_odom>true</publish_odom>
+                <max_wheel_acceleration>5.0</max_wheel_acceleration>
+                <!-- Odometry source, 0 for ENCODER, 1 for WORLD, defaults to WORLD -->
+                <xacro:if value="${odometry_source == 'world'}">
+                    <odometry_source>1</odometry_source>
+                </xacro:if>
+                <xacro:if value="${odometry_source == 'encoder'}">
+                    <odometry_source>0</odometry_source>
+                </xacro:if>
+            </plugin>
         </gazebo>
         <!--............................... IMU PLUGIN ..................................... -->
@@ -94,5 +125,5 @@
                         <width>1024</width>
                         <height>1024</height>
-                        <format>BGR8</format>
+                        <format>R8G8B8</format>
                     </image>
                     <clip>
@@ -120,5 +151,5 @@
                         <width>1024</width>
                         <height>1024</height>
-                        <format>BGR8</format>
+                        <format>R8G8B8</format>
                     </image>
                     <clip>

File: src/agv_with_arm/urdf/agv/robot.urdf.xacro (robot description, xacro)
@@ -13,8 +13,8 @@
             <origin xyz="0.0 0.0 0.0" rpy="0.0 0.0 0.0" />
         </joint>
+        <!-- 控制器 -->
+        <xacro:include filename="$(find agv_with_arm)/urdf/arm/ros2_control.xacro" />
+        <xacro:arm_ros2_control />
     </xacro:if>
-    <!-- 控制器 -->
-    <xacro:include filename="$(find agv_with_arm)/urdf/agv/ros2_control.xacro" />
-    <xacro:agv_sim_ros2_control arm_enabled="$(arg arm_enabled)"/>
     <!-- gazebo 仿真配置 -->
     <xacro:include filename="$(find agv_with_arm)/urdf/agv/gazebo_sensor.xacro"/>

File: src/agv_with_arm/urdf/agv/robot_core.xacro (robot description, xacro)
@@ -2,9 +2,9 @@
 <robot xmlns:xacro="http://www.ros.org/wiki/xacro" name="agv_with_arm">
     <!--................................ XACRO CONSTANTS .............................. -->
-    <xacro:property name="chassis_mass" value="1"/>
+    <xacro:property name="chassis_mass" value="70"/>
     <xacro:property name="chassis_length" value="0.9"/>
     <xacro:property name="chassis_width" value="0.64"/>
     <xacro:property name="chassis_height" value="0.19"/>
-    <xacro:property name="traction_wheel_mass" value="0.5"/>
+    <xacro:property name="traction_wheel_mass" value="1"/>
     <xacro:property name="traction_wheel_base" value="0.88"/>
     <xacro:property name="traction_max_wheel_torque" value="20000"/>
@@ -15,5 +15,5 @@
     <xacro:property name="trolley_wheel_radius" value="0.06"/>
     <!-- a small constant -->
-    <xacro:property name="eps" value="0.001"/>
+    <xacro:property name="eps" value="0.002"/>
     <xacro:property name="traction_wheel_radius" value="0.1"/>
     <xacro:property name="traction_wheel_width" value="0.05"/>
@@ -30,8 +30,13 @@
     <xacro:arg name="robot_namespace" default=""/>
     <xacro:arg name="wheel_odom_topic" default="odom" />
+    <xacro:arg name="camera_enabled" default="false" />
+    <xacro:arg name="stereo_camera_enabled" default="false" />
+    <xacro:arg name="two_d_lidar_enabled" default="false" />
     <xacro:arg name="publish_wheel_odom_tf" default="true" />
     <xacro:arg name="conveyor_enabled" default="false"/>
     <xacro:arg name="ground_truth_frame" default="map"/>
-    <xacro:arg name="sim_ign" default="true" />
+    <xacro:arg name="sim_gazebo" default="false" />
+    <xacro:arg name="sim_ign" default="false" />
+    <xacro:arg name="sim_gz" default="false" />
     <xacro:arg name="odometry_source" default="world" />
     <xacro:property name="odometry_source" value="$(arg odometry_source)"/>

File: src/agv_with_arm/urdf/agv/ros2_control.xacro (robot description, xacro)
@@ -6,4 +6,5 @@
                 <plugin>gazebo_ros2_control/GazeboSystem</plugin>
             </hardware>
+            <!-- 使用ros2_control来控制小车 -->
             <joint name="middle_left_wheel_joint">
                 <command_interface name="velocity">
