Commit message: 实现gazebo+moveit2+agv的小车和机械臂控制

File: src/agv_with_arm/urdf/agv/robot.urdf.xacro (robot description, xacro)
@@ -3,6 +3,7 @@
     <xacro:arg name="arm_enabled" default="true"/>
     <xacro:arg name="robot_namespace" default="agv_with_arm"/>
+    <xacro:arg name="initial_positions_file" default="$(find agv_with_arm)/config/initial_positions.yaml" />
     <!-- robot description -->
-    <xacro:include filename="robot_core.xacro" />
+    <xacro:include filename="$(find agv_with_arm)/urdf/agv/robot_core.xacro" />
     <!-- 机械臂 -->
     <xacro:if value="$(arg arm_enabled)">
@@ -14,6 +15,6 @@
         </joint>
         <!-- 控制器 -->
-        <xacro:include filename="$(find agv_with_arm)/urdf/arm/ros2_control.xacro" />
-        <xacro:arm_ros2_control />
+        <xacro:include filename="$(find agv_with_arm)/urdf/arm/aubo_i5.ros2_control.xacro" />
+        <xacro:aubo_i5_ros2_control name="GazeboSystem" initial_positions_file="$(arg initial_positions_file)"/>
     </xacro:if>
     <!-- gazebo 仿真配置 -->

File: src/agv_with_arm/urdf/arm/aubo.gazebo.xacro (robot description, xacro)
@@ -205,9 +205,93 @@
           <limit lower="-6.28" upper="6.28" effort="10" velocity="1.5" />
      </joint>
-     <!-- <link name="world" />
-     <joint name="world_joint" type="fixed">
-          <parent link="world" />
-          <child link = "arm_base_link" />
-          <origin xyz="0.0 0.0 0.0" rpy="0.0 0.0 0.0" />
-     </joint> -->
+     <!-- panda_hand -->
+     <joint name="panda_hand_joint" type="fixed">
+          <parent link="wrist3_Link"/>
+          <child link="panda_hand"/>
+          <origin rpy="0 0 0" xyz="0 0 0"/>
+     </joint>
+     <link name="panda_hand">
+          <inertial>
+               <mass value="0.73"/>
+               <origin rpy="0 0 0" xyz="0 0.0015244 0.0275912"/>
+               <inertia ixx="0.00278560230025" ixy="0.0" ixz="0.0" iyy="0.000400033405336" iyz="0.0" izz="0.00256378041832"/>
+          </inertial>
+          <visual>
+               <origin rpy="0 0 0" xyz="0 0 0"/>
+               <geometry>
+                    <mesh filename="file://$(find panda_ros2_gazebo)/meshes/visual/hand.dae"/>
+               </geometry>
+               <material name="">
+                    <color rgba="1 1 1 1"/>
+               </material>
+          </visual>
+          <collision>
+               <origin rpy="0 0 0" xyz="0 0 0"/>
+               <geometry>
+                    <mesh filename="file://$(find panda_ros2_gazebo)/meshes/collision/hand.stl"/>
+               </geometry>
+          </collision>
+     </link>
+     <!-- panda_leftfinger -->
+     <link name="panda_leftfinger">
+          <inertial>
+               <mass value="0.1"/>
+               <origin rpy="0 0 0" xyz="0 0.0145644 0.0227941"/>
+               <inertia ixx="3.01220925051e-05" ixy="0.0" ixz="0.0" iyy="2.95873808038e-05" iyz="0.0" izz="6.95125211657e-06"/>
+          </inertial>
+          <visual>
+               <origin rpy="0 0 0" xyz="0 0 0"/>
+               <geometry>
+                    <mesh filename="file://$(find panda_ros2_gazebo)/meshes/visual/finger.dae"/>
+               </geometry>
+               <material name="">
+                    <color rgba="1 1 1 1"/>
+               </material>
+          </visual>
+          <collision>
+               <origin rpy="0 0 0" xyz="0 0 0"/>
+               <geometry>
+                    <mesh filename="file://$(find panda_ros2_gazebo)/meshes/collision/finger.stl"/>
+               </geometry>
+          </collision>
+     </link>
+     <!-- panda_rightfinger -->
+     <link name="panda_rightfinger">
+          <inertial>
+               <mass value="0.1"/>
+               <origin rpy="0 0 3.14159265359" xyz="0 0.0145644 0.0227941"/>
+               <inertia ixx="3.01220925051e-05" ixy="0.0" ixz="0.0" iyy="2.95873808038e-05" iyz="0.0" izz="6.95125211657e-06"/>
+          </inertial>
+          <visual>
+               <origin rpy="0 0 3.14159265359" xyz="0 0 0"/>
+               <geometry>
+                    <mesh filename="file://$(find panda_ros2_gazebo)/meshes/visual/finger.dae"/>
+               </geometry>
+               <material name="">
+                    <color rgba="1 1 1 1"/>
+               </material>
+          </visual>
+          <collision>
+               <origin rpy="0 0 3.14159265359" xyz="0 0 0"/>
+               <geometry>
+                    <mesh filename="file://$(find panda_ros2_gazebo)/meshes/collision/finger.stl"/>
+               </geometry>
+          </collision>
+     </link>
+     <joint name="panda_finger_joint1" type="prismatic">
+          <parent link="panda_hand"/>
+          <child link="panda_leftfinger"/>
+          <origin rpy="0 0 0" xyz="0 0 0.0584"/>
+          <axis xyz="0 1 0"/>
+          <limit effort="20" lower="-0.001" upper="0.04" velocity="0.3"/>
+          <dynamics damping="1.0" friction="1.0"/>
+     </joint>
+     <joint name="panda_finger_joint2" type="prismatic">
+          <parent link="panda_hand"/>
+          <child link="panda_rightfinger"/>
+          <origin rpy="0 0 0" xyz="0 0 0.0584"/>
+          <axis xyz="0 -1 0"/>
+          <limit effort="20" lower="-0.001" upper="0.04" velocity="0.3"/>
+          <dynamics damping="1.0" friction="1.0"/>
+     </joint>
 </robot>
