Commit message: README优化

File: src/agv_with_arm/urdf/arm/aubo.gazebo.xacro (robot description, xacro)
@@ -295,3 +295,9 @@
           <dynamics damping="1.0" friction="1.0"/>
      </joint>
+     <link name="world"/>
+     <joint name="world_joint" type="fixed">
+          <parent link="world" />
+          <child link = "arm_base_link" />
+          <origin xyz="0.0 0.0 0.0" rpy="0.0 0.0 0.0" />
+     </joint>
 </robot>
